Commit message: noetic branch

File: racebot_description/urdf/ackermann/racecar.xacro (robot description, xacro)
@@ -39,5 +39,5 @@
     <parent link="base_link" />
     <child link="base_inertia" />
-  </joint>
+    </joint>
     <link name="left_steering_hinge">
         <visual>

File: racebot_description/urdf/tianracer/tianracer.xacro (robot description, xacro)
@@ -38,5 +38,5 @@
     <parent link="base_link" />
     <child link="base_inertia" />
-  </joint>
+    </joint>
     <link name="left_steering_hinge">
         <visual>
@@ -100,9 +100,9 @@
         <limit effort="10" velocity="1000" />
     </joint>
-     <xacro:wheel_transmission name="left_front_wheel" />
+    <xacro:wheel_transmission name="left_front_wheel" />
 <link name="right_steering_hinge">
         <visual>
             <geometry>
-                 <cylinder radius="0.01" length="0.005" />
+                <cylinder radius="0.01" length="0.005" />
             </geometry>
             <origin xyz="0 0 0" rpy="1.57 0 0" />
@@ -131,5 +131,5 @@
     </joint>
     <xacro:steering_hinge_transmission name="right_steering_hinge" />
-     <link name="right_front_wheel">
+    <link name="right_front_wheel">
         <visual>
             <geometry>
@@ -342,4 +342,4 @@
         <axis xyz="0 0 1" />
     </joint>
-  <xacro:include filename="$(find racebot_description)/urdf/ackermann/racecar.gazebo" />
+    <xacro:include filename="$(find racebot_description)/urdf/ackermann/racecar.gazebo" />
 </robot>

File: racebot_description/urdf/twist/macros.xacro (robot description, xacro)
@@ -26,5 +26,5 @@
   </transmission>
 </xacro:macro> -->
- <!-- motors and transmissions for the two rear wheels -->
+  <!-- motors and transmissions for the two rear wheels -->
   <transmission name="tran1">
     <type>transmission_interface/SimpleTransmission</type>

File: racebot_description/urdf/twist/racecar.xacro (robot description, xacro)
@@ -36,5 +36,5 @@
         <origin xyz="0 0 0.032" />
     </joint>
-       <link name="left_steering_hinge">
+    <link name="left_steering_hinge">
         <visual>
             <geometry>
@@ -99,5 +99,5 @@
         <visual>
             <geometry>
-                 <cylinder radius="0.01" length="0.005" />
+                <cylinder radius="0.01" length="0.005" />
             </geometry>
             <origin xyz="0 0 0" rpy="1.57 0 0" />
@@ -125,5 +125,5 @@
         <limit lower="-0.6" upper="0.6" effort="2.0" velocity="100.0"/>
     </joint>
-     <link name="right_front_wheel">
+    <link name="right_front_wheel">
         <visual>
             <geometry>
@@ -212,4 +212,4 @@
         <limit effort="10" velocity="1000" />
     </joint>
-  <xacro:include filename="$(find racebot_description)/urdf/twist/racecar.gazebo" />
+    <xacro:include filename="$(find racebot_description)/urdf/twist/racecar.gazebo" />
 </robot>
